Commit message: Visual potential field with different risk functions

File: urdf/quadrotor_front_camera.gazebo.xacro (robot description, xacro)
@@ -24,10 +24,10 @@
     <parent link="base_link"/>
     <child link="front_camera_link"/>
-    <origin xyz="0.05 0 -0.15" rpy="0 0.2 0"/>
+    <origin xyz="0.25 0 0" rpy="0 0 0"/>
   </joint>
   <gazebo reference="front_camera_link">
     <sensor type="camera" name="front_rgb_camera">
       <always_on>true</always_on>
-      <update_rate>60</update_rate>
+      <update_rate>30</update_rate>
       <camera>
         <horizontal_fov>1.3962634</horizontal_fov>
@@ -49,5 +49,5 @@
         <frameName>front_camera_link</frameName>
         <alwaysOn>true</alwaysOn>
-        <updateRate>60</updateRate>
+        <updateRate>30</updateRate>
       </plugin>
     </sensor>

Commit message: Cleaned up structure oof the folders

File: urdf/quadrotor_front_camera.gazebo.xacro (robot description, xacro)
@@ -24,5 +24,5 @@
     <parent link="base_link"/>
     <child link="front_camera_link"/>
-    <origin xyz="0.25 0 0" rpy="0 0 0"/>
+    <origin xyz="0.25 0 -0.05" rpy="0 0 0"/>
   </joint>
   <gazebo reference="front_camera_link">
